File: hardware/logicboard/p2d-001.sch (EAGLE design)
At the start: 60 parts, among them IC1 74LS06N, IC2 4066N, IC3 MAX3468CPA, J1 MKR, J2 GPIO, J3 Vcc, J4 RLY, J5 SPI, K1 G5V1, T1 2SC1815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

Commit message: Try. Error.
Parts:
- removed SV4: (no value), con-ml:ML20LE
- added JP7: (no value), pinhead:PINHD-2X10
Connections:
- net GND: now also JP7.1, JP7.15, JP7.5
- net LED0: now also JP7.7
- net MIRTN: now also JP7.11
- net MISND: now also JP7.9
- net MORTN: now also JP7.17
- net MOSND: now also JP7.13
- net RST: now also JP7.3
- net VCC: now also JP7.19
Changed lines of the file:
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@@
 <part name="V+1" library="wirepad" library_urn="urn:adsk.eagle:library:412" deviceset="SMD2" device="" package3d_urn="urn:adsk.eagle:package:30839/1"/>
 <part name="VIN1" library="wirepad" library_urn="urn:adsk.eagle:library:412" deviceset="SMD2" device="" package3d_urn="urn:adsk.eagle:package:30839/1"/>
-<part name="SV4" library="con-ml" library_urn="urn:adsk.eagle:library:164" deviceset="ML20LE" device="" package3d_urn="urn:adsk.eagle:package:8685/1"/>
+<part name="JP7" library="pinhead" library_urn="urn:adsk.eagle:library:325" deviceset="PINHD-2X10" device="" package3d_urn="urn:adsk.eagle:package:22405/2"/>
 </parts>
 <sheets>
@@
 <attribute name="VALUE" x="136.398" y="105.283" size="1.778" layer="96" rot="R270"/>
 </instance>
-<instance part="SV4" gate="-1" x="314.96" y="91.44" smashed="yes">
-<attribute name="NAME" x="317.5" y="90.678" size="1.778" layer="95"/>
-<attribute name="VALUE" x="314.706" y="88.519" size="1.778" layer="96"/>
-</instance>
-<instance part="SV4" gate="-2" x="314.96" y="86.36" smashed="yes">
-<attribute name="NAME" x="317.5" y="85.598" size="1.778" layer="95"/>
-<attribute name="VALUE" x="314.706" y="83.439" size="1.778" layer="96"/>
-</instance>
-<instance part="SV4" gate="-3" x="314.96" y="81.28" smashed="yes">
-<attribute name="NAME" x="317.5" y="80.518" size="1.778" layer="95"/>
-<attribute name="VALUE" x="314.706" y="78.359" size="1.778" layer="96"/>
-</instance>
-<instance part="SV4" gate="-4" x="314.96" y="76.2" smashed="yes">
-<attribute name="NAME" x="317.5" y="75.438" size="1.778" layer="95"/>
-<attribute name="VALUE" x="314.706" y="73.279" size="1.778" layer="96"/>
-</instance>
-<instance part="SV4" gate="-5" x="314.96" y="71.12" smashed="yes">
-<attribute name="NAME" x="317.5" y="70.358" size="1.778" layer="95"/>
-<attribute name="VALUE" x="314.706" y="68.199" size="1.778" layer="96"/>
-</instance>
-<instance part="SV4" gate="-6" x="314.96" y="66.04" smashed="yes">
-<attribute name="NAME" x="317.5" y="65.278" size="1.778" layer="95"/>
-<attribute name="VALUE" x="314.706" y="63.119" size="1.778" layer="96"/>
-</instance>
-<instance part="SV4" gate="-7" x="314.96" y="60.96" smashed="yes">
-<attribute name="NAME" x="317.5" y="60.198" size="1.778" layer="95"/>
-<attribute name="VALUE" x="314.706" y="58.039" size="1.778" layer="96"/>
-</instance>
-<instance part="SV4" gate="-8" x="314.96" y="55.88" smashed="yes">
-<attribute name="NAME" x="317.5" y="55.118" size="1.778" layer="95"/>
-<attribute name="VALUE" x="314.706" y="52.959" size="1.778" layer="96"/>
-</instance>
-<instance part="SV4" gate="-9" x="314.96" y="50.8" smashed="yes">
-<attribute name="NAME" x="317.5" y="50.038" size="1.778" layer="95"/>
-<attribute name="VALUE" x="314.706" y="47.879" size="1.778" layer="96"/>
-</instance>
-<instance part="SV4" gate="-10" x="314.96" y="45.72" smashed="yes">
-<attribute name="NAME" x="317.5" y="44.958" size="1.778" layer="95"/>
-<attribute name="VALUE" x="314.706" y="42.799" size="1.778" layer="96"/>
-</instance>
-<instance part="SV4" gate="-11" x="335.28" y="91.44" smashed="yes">
-<attribute name="NAME" x="337.82" y="90.678" size="1.778" layer="95"/>
-<attribute name="VALUE" x="335.026" y="88.519" size="1.778" layer="96"/>
-</instance>
-<instance part="SV4" gate="-12" x="335.28" y="86.36" smashed="yes">
-<attribute name="NAME" x="337.82" y="85.598" size="1.778" layer="95"/>
-<attribute name="VALUE" x="335.026" y="83.439" size="1.778" layer="96"/>
-</instance>
-<instance part="SV4" gate="-13" x="335.28" y="81.28" smashed="yes">
-<attribute name="NAME" x="337.82" y="80.518" size="1.778" layer="95"/>
-<attribute name="VALUE" x="335.026" y="78.359" size="1.778" layer="96"/>
-</instance>
-<instance part="SV4" gate="-14" x="335.28" y="76.2" smashed="yes">
-<attribute name="NAME" x="337.82" y="75.438" size="1.778" layer="95"/>
-<attribute name="VALUE" x="335.026" y="73.279" size="1.778" layer="96"/>
-</instance>
-<instance part="SV4" gate="-15" x="335.28" y="71.12" smashed="yes">
-<attribute name="NAME" x="337.82" y="70.358" size="1.778" layer="95"/>
-<attribute name="VALUE" x="335.026" y="68.199" size="1.778" layer="96"/>
-</instance>
-<instance part="SV4" gate="-16" x="335.28" y="66.04" smashed="yes">
-<attribute name="NAME" x="337.82" y="65.278" size="1.778" layer="95"/>
-<attribute name="VALUE" x="335.026" y="63.119" size="1.778" layer="96"/>
-</instance>
-<instance part="SV4" gate="-17" x="335.28" y="60.96" smashed="yes">
-<attribute name="NAME" x="337.82" y="60.198" size="1.778" layer="95"/>
-<attribute name="VALUE" x="335.026" y="58.039" size="1.778" layer="96"/>
-</instance>
-<instance part="SV4" gate="-18" x="335.28" y="55.88" smashed="yes">
-<attribute name="NAME" x="337.82" y="55.118" size="1.778" layer="95"/>
-<attribute name="VALUE" x="335.026" y="52.959" size="1.778" layer="96"/>
-</instance>
-<instance part="SV4" gate="-19" x="335.28" y="50.8" smashed="yes">
-<attribute name="NAME" x="337.82" y="50.038" size="1.778" layer="95"/>
-<attribute name="VALUE" x="335.026" y="47.879" size="1.778" layer="96"/>
-</instance>
-<instance part="SV4" gate="-20" x="335.28" y="45.72" smashed="yes">
-<attribute name="NAME" x="337.82" y="44.958" size="1.778" layer="95"/>
-<attribute name="VALUE" x="335.026" y="42.799" size="1.778" layer="96"/>
+<instance part="JP7" gate="A" x="279.4" y="66.04" smashed="yes">
+<attribute name="NAME" x="273.05" y="79.375" size="1.778" layer="95"/>
+<attribute name="VALUE" x="273.05" y="48.26" size="1.778" layer="96"/>
 </instance>
 </instances>
@@
 <junction x="226.06" y="43.18"/>
 </segment>
+<segment>
+<pinref part="JP7" gate="A" pin="1"/>
+<wire x1="276.86" y1="76.2" x2="269.24" y2="76.2" width="0.1524" layer="91"/>
+<label x="269.24" y="76.2" size="0.8128" layer="95" rot="R180" xref="yes"/>
+</segment>
+<segment>
+<pinref part="JP7" gate="A" pin="5"/>
+<wire x1="276.86" y1="71.12" x2="269.24" y2="71.12" width="0.1524" layer="91"/>
+<label x="269.24" y="71.12" size="0.8128" layer="95" rot="R180" xref="yes"/>
+</segment>
+<segment>
+<pinref part="JP7" gate="A" pin="15"/>
+<wire x1="276.86" y1="58.42" x2="269.24" y2="58.42" width="0.1524" layer="91"/>
+<label x="269.24" y="58.42" size="0.8128" layer="95" rot="R180" xref="yes"/>
+</segment>
 </net>
 <net name="VCC" class="2">
@@
 <label x="177.8" y="27.94" size="0.8128" layer="95" xref="yes"/>
 </segment>
+<segment>
+<pinref part="JP7" gate="A" pin="19"/>
+<wire x1="276.86" y1="53.34" x2="269.24" y2="53.34" width="0.1524" layer="91"/>
+<label x="269.24" y="53.34" size="0.8128" layer="95" rot="R180" xref="yes"/>
+</segment>
 </net>
 <net name="RLYSNK" class="0">
@@
 <label x="340.36" y="116.84" size="0.8128" layer="95" rot="MR0" xref="yes"/>
 </segment>
+<segment>
+<pinref part="JP7" gate="A" pin="3"/>
+<wire x1="276.86" y1="73.66" x2="269.24" y2="73.66" width="0.1524" layer="91"/>
+<label x="269.24" y="73.66" size="0.8128" layer="95" rot="R180" xref="yes"/>
+</segment>
 </net>
 <net name="THS" class="0">
@@
 <label x="101.6" y="33.02" size="0.8128" layer="95" xref="yes"/>
 <pinref part="R4" gate="G$1" pin="2"/>
+</segment>
+<segment>
+<pinref part="JP7" gate="A" pin="7"/>
+<wire x1="276.86" y1="68.58" x2="269.24" y2="68.58" width="0.1524" layer="91"/>
+<label x="269.24" y="68.58" size="0.8128" layer="95" rot="R180" xref="yes"/>
 </segment>
 </net>
@@
 <junction x="208.28" y="116.84"/>
 </segment>
+<segment>
+<pinref part="JP7" gate="A" pin="11"/>
+<wire x1="276.86" y1="63.5" x2="269.24" y2="63.5" width="0.1524" layer="91"/>
+<label x="269.24" y="63.5" size="0.8128" layer="95" rot="R180" xref="yes"/>
+</segment>
 </net>
 <net name="MI" class="0">
@@
 <label x="213.36" y="124.46" size="0.8128" layer="95" xref="yes"/>
 </segment>
+<segment>
+<pinref part="JP7" gate="A" pin="9"/>
+<wire x1="276.86" y1="66.04" x2="269.24" y2="66.04" width="0.1524" layer="91"/>
+<label x="269.24" y="66.04" size="0.8128" layer="95" rot="R180" xref="yes"/>
+</segment>
 </net>
 <net name="N$5" class="0">
@@
 <label x="195.58" y="33.02" size="0.8128" layer="95" xref="yes"/>
 </segment>
+<segment>
+<pinref part="JP7" gate="A" pin="17"/>
+<wire x1="276.86" y1="55.88" x2="269.24" y2="55.88" width="0.1524" layer="91"/>
+<label x="269.24" y="55.88" size="0.8128" layer="95" rot="R180" xref="yes"/>
+</segment>
 </net>
 <net name="MOSND" class="0">
@@
 <label x="195.58" y="38.1" size="0.8128" layer="95" xref="yes"/>
 </segment>
-</net>
+<segment>
+<pinref part="JP7" gate="A" pin="13"/>
+<wire x1="276.86" y1="60.96" x2="269.24" y2="60.96" width="0.1524" layer="91"/>
+<label x="269.24" y="60.96" size="0.8128" layer="95" rot="R180" xref="yes"/>
+</segment>
+</net>

Commit message: Routing test.
Parts:
- added A, B, V/2, VO: (no value), wirepad:SMD2
- SV3: device con-ml:ML14E -> pinhead:PINHD-2X7
- renumbered JP7 to SV2, V+1 to RX, VIN1 to DMXRX
Connections:
- net D7GATE: now also SV3.11; no longer SV3-11.S
- net DTCT0: now also SV3.6; no longer SV3-6.S
- net DTCT1: now also SV3.8; no longer SV3-8.S
- net DTCT2: now also SV3.10; no longer SV3-10.S
- net DTCT3: now also SV3.12; no longer SV3-12.S
- net GND: now also SV3.5; no longer SV3-5.S
- net GPIO0: now also SV3.2; no longer SV3-2.S
- net GPIO1: now also SV3.4; no longer SV3-4.S
- net RX: now also SV3.1; no longer SV3-1.S
- net SCL: now also SV3.9; no longer SV3-9.S
- net SDA: now also SV3.7; no longer SV3-7.S
- net THS: now also SV3.14; no longer SV3-14.S
- net TX: now also SV3.3; no longer SV3-3.S
- net VCC: now also SV3.13; no longer SV3-13.S
- net VCC/2: now also V/2.P
- net VOUT: now also VO.P
- net VOUTRAW: now also B.P
- net VOUTRAW2: now also A.P
Other:
- moved on the sheet: D2, F1, K1, R1, R2, T1, U1

Commit message: First try.
Parts:
- JP03SELFTERMINATE: device pinhead:PINHD-1X2 -> pinhead:PINHD-1X2/90
Changed lines of the file:
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@@
 <part name="R700" library="resistor" library_urn="urn:adsk.eagle:library:348" deviceset="R-EU_" device="0204/5" package3d_urn="urn:adsk.eagle:package:23488/1" value="120"/>
 <part name="SUPPLY10" library="supply2" deviceset="GND" device=""/>
-<part name="JP03SELFTERMINATE" library="pinhead" library_urn="urn:adsk.eagle:library:325" deviceset="PINHD-1X2" device="" package3d_urn="urn:adsk.eagle:package:22435/2"/>
+<part name="JP03SELFTERMINATE" library="pinhead" library_urn="urn:adsk.eagle:library:325" deviceset="PINHD-1X2" device="/90" package3d_urn="urn:adsk.eagle:package:22437/2"/>
 <part name="SUPPLY14" library="supply2" deviceset="GND" device=""/>
 <part name="IC1" library="74xx-us" library_urn="urn:adsk.eagle:library:88" deviceset="74*06" device="N" package3d_urn="urn:adsk.eagle:package:16407/2" technology="LS"/>

Commit message: Looks ok.
Parts:
- renumbered JP03SELFTERMINATE to JP10, R700 to R10
Changed lines of the file:
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@@
 <part name="X2" library="con-neutrik_ag" library_urn="urn:adsk.eagle:library:166" deviceset="NC3" device="MBH" package3d_urn="urn:adsk.eagle:package:8841/1"/>
 <part name="IC3" library="maxim" library_urn="urn:adsk.eagle:library:269" deviceset="MAX34*" device="PA" package3d_urn="urn:adsk.eagle:package:29519/2" technology="68C"/>
-<part name="R700" library="resistor" library_urn="urn:adsk.eagle:library:348" deviceset="R-EU_" device="0204/5" package3d_urn="urn:adsk.eagle:package:23488/1" value="120"/>
+<part name="R10" library="resistor" library_urn="urn:adsk.eagle:library:348" deviceset="R-EU_" device="0204/5" package3d_urn="urn:adsk.eagle:package:23488/1" value="120"/>
 <part name="SUPPLY10" library="supply2" deviceset="GND" device=""/>
-<part name="JP03SELFTERMINATE" library="pinhead" library_urn="urn:adsk.eagle:library:325" deviceset="PINHD-1X2" device="/90" package3d_urn="urn:adsk.eagle:package:22437/2"/>
+<part name="JP10" library="pinhead" library_urn="urn:adsk.eagle:library:325" deviceset="PINHD-1X2" device="/90" package3d_urn="urn:adsk.eagle:package:22437/2"/>
 <part name="SUPPLY14" library="supply2" deviceset="GND" device=""/>
 <part name="IC1" library="74xx-us" library_urn="urn:adsk.eagle:library:88" deviceset="74*06" device="N" package3d_urn="urn:adsk.eagle:package:16407/2" technology="LS"/>
@@
 <attribute name="VALUE" x="167.64" y="48.26" size="1.778" layer="96"/>
 </instance>
-<instance part="R700" gate="G$1" x="226.06" y="66.04" smashed="yes">
+<instance part="R10" gate="G$1" x="226.06" y="66.04" smashed="yes">
 <attribute name="NAME" x="226.06" y="68.58" size="1.778" layer="95" align="bottom-center"/>
 <attribute name="VALUE" x="226.06" y="63.5" size="1.778" layer="96" align="top-center"/>
 </instance>
 <instance part="SUPPLY10" gate="GND" x="198.12" y="48.26" smashed="yes"/>
-<instance part="JP03SELFTERMINATE" gate="G$1" x="238.76" y="63.5" smashed="yes">
+<instance part="JP10" gate="G$1" x="238.76" y="63.5" smashed="yes">
 <attribute name="NAME" x="232.41" y="69.215" size="1.778" layer="95"/>
 <attribute name="VALUE" x="232.41" y="58.42" size="1.778" layer="96"/>
@@
 </segment>
 <segment>
-<pinref part="R700" gate="G$1" pin="1"/>
+<pinref part="R10" gate="G$1" pin="1"/>
 <wire x1="220.98" y1="66.04" x2="218.44" y2="66.04" width="0.1524" layer="91"/>
 <label x="218.44" y="66.04" size="0.8128" layer="95" rot="R180" xref="yes"/>
@@
 </segment>
 <segment>
-<pinref part="JP03SELFTERMINATE" gate="G$1" pin="2"/>
+<pinref part="JP10" gate="G$1" pin="2"/>
 <wire x1="236.22" y1="63.5" x2="218.44" y2="63.5" width="0.1524" layer="91"/>
 <label x="218.44" y="63.5" size="0.8128" layer="95" rot="R180" xref="yes"/>
@@
 <net name="N$1" class="0">
 <segment>
-<pinref part="JP03SELFTERMINATE" gate="G$1" pin="1"/>
-<pinref part="R700" gate="G$1" pin="2"/>
+<pinref part="JP10" gate="G$1" pin="1"/>
+<pinref part="R10" gate="G$1" pin="2"/>
 <wire x1="236.22" y1="66.04" x2="231.14" y2="66.04" width="0.1524" layer="91"/>
 </segment>
